Commit message: Added model into main page in a small square

File: gh360_gui/gh360 ThreeJS model/urdf/gh360.urdf (robot description, URDF)
Before this commit: robot multipleshapes, 13 links, 12 joints
Joints:
- joint base_joint: origin xyz=0 0.0 0 rpy=0 1.571 1.571 -> xyz=0 0.0 0 rpy=0 1.571 0
- joint forearm_roll: origin xyz=0.000 -0.074 -0.041 rpy=0 0 0 -> xyz=0.000 -0.074 -0.041 rpy=1.5 0 0
- joint upperarm_roll: origin xyz=0.001 -0.107 -0.014 rpy=0 0 0 -> xyz=0.001 -0.107 -0.014 rpy=0 -1.5 0
- joint wrist_pitch: origin xyz=0.0 -0.169 0.0 rpy=0 0 0 -> xyz=0.0 -0.169 0.0 rpy=0 3.125 0

Commit message: .

File: gh360_gui/gh360 ThreeJS model/urdf/gh360.urdf (robot description, URDF)
Before this commit: robot multipleshapes, 13 links, 12 joints
Links:
- removed link eef

Commit message: fixed model forearm rotation

File: gh360_gui/gh360 ThreeJS model/urdf/gh360.urdf (robot description, URDF)
Before this commit: robot multipleshapes, 12 links, 12 joints
Joints:
- joint forearm_roll: origin xyz=0.000 -0.074 -0.041 rpy=1.5 0 0 -> xyz=0.000 -0.074 -0.041 rpy=0 0 0

Commit message: UI breakpoint now correctly works for bigger laptop screens. Open and closeable navbar, model now takes up full height. Need to display the camera

File: gh360_gui/gh360 ThreeJS model/urdf/gh360.urdf (robot description, URDF)
Before this commit: robot multipleshapes, 12 links, 12 joints
Joints:
- joint base_joint: origin xyz=0 0.0 0 rpy=0 1.571 0 -> xyz=0 0.0 0 rpy=0 1 0
- joint forearm_roll: origin xyz=0.000 -0.074 -0.041 rpy=1.5 0 0 -> xyz=0.000 -0.074 -0.041 rpy=0 0 0

Commit message: Move arm page changed to show slider positions rather than message positions

File: gh360_gui/gh360 ThreeJS model/urdf/gh360.urdf (robot description, URDF)
Before this commit: robot multipleshapes, 12 links, 12 joints
Joints:
- joint upperarm_roll: origin xyz=0.001 -0.107 -0.014 rpy=0 -1.5 0 -> xyz=0.001 -0.107 -0.014 rpy=0 0 0
