Commit message: .

File: gh360_gui/public/gh360-threejs-model/urdf/gh360.urdf (robot description, URDF)
Before this commit: robot multipleshapes, 12 links, 12 joints
Joints:
- joint wrist_pitch: origin xyz=0.0 -0.169 0.0 rpy=0 3.125 0 -> xyz=0.0 -0.169 0.0 rpy=0 0 0

File: gh360_gui/public/gh360-threejs-model/urdf/gh360_ghost.urdf (robot description, URDF)
Before this commit: robot multipleshapes, 12 links, 12 joints
Joints:
- joint wrist_pitch: origin xyz=0.0 -0.169 0.0 rpy=0 3.125 0 -> xyz=0.0 -0.169 0.0 rpy=0 0 0
